File: project_02/ArcadeMachine.brd (EAGLE design)
At the start: 5 parts, among them U1 POCKETBEAGLE, U2 0.56_HEX_BACKPACK, U3 BUZZER

Commit message: Finished project
Parts:
- added C1: 1uF, ArcadeMachine:SPARKFUN-CAPACITORS_0603-CAP
- added FUD1, FUD2, FUD3: FIDUCIAL, ArcadeMachine:FIDUCIAL_40MIL
- added R3, R4, R5, R6: 1K, ArcadeMachine:R0603
- added SW1, SW2, SW3, SW4: LED_TACTILE_BUTTON, ArcadeMachine:LED_TACTILE_BUTTON
- added SW5: ROTARY_SWITCH, ArcadeMachine:ROTARY_SWITCH
- added U4: TPD4S012_DRY_6, ArcadeMachine:BEAGLEBONE_BLUE_DRY6
- added X1: (no value), ArcadeMachine:GHI2_USB_HOST_HORIZONTAL_W/CHASSIS_GND
- moved U3 184.6 mm to (30.5, 104.1)
- moved R2 157.4 mm to (38.1, 59.7)
- moved R1 150.3 mm to (27.9, 59.7)
- moved U2 144.4 mm to (34.9, 76.8)
- moved U1 105.2 mm to (8.13, 55.1), flipped to the bottom, turned to 180 degrees
Connections:
- new net BUZZER: U1.54, U3.+
- new net LED_0: SW1.5, U1.66
- new net LED_1: SW2.5, U1.56
- new net LED_2: SW3.5, U1.70
- new net LED_3: SW4.5, U1.60
- new net PB_0: R3.1, SW1.1, SW1.3, U1.64
- new net PB_1: R4.1, SW2.1, SW2.3, U1.53
- new net PB_2: R6.1, SW3.1, SW3.3, U1.68
- new net PB_3: R5.1, SW4.1, SW4.3, U1.58
- new net SW_0: SW5.1, U1.40
- new net SW_1: SW5.2, U1.42
- new net SW_2: SW5.3, U1.44
- new net SW_3: SW5.4, U1.46
- new net SW_4: SW5.5, U1.38
- new net USBC.D+: U1.9, U4.2, X1.3
- new net USBC.D-: U1.11, U4.1, X1.2
- new net USB_DC: C1.1, U4.6, X1.1
- new net VOUT: U1.49
- net GND: now also C1.2, SW1.2, SW1.4, SW1.6, SW2.2, SW2.4, SW2.6, SW3.2, SW3.4, SW3.6, SW4.2, SW4.4, SW4.6, SW5.C, U3.-, U4.4, X1.4
- net VDD_3P3V: now also R3.2, R4.2, R5.2, R6.2
- net VDD_5V: no longer U1.49
Routing:
- net SW_1: track 0.00 -> 172.7 mm
- net SW_2: track 0.00 -> 166.3 mm
- net SW_3: track 0.00 -> 159.8 mm
- net BUZZER: track 0.00 -> 118.7 mm
- net SW_0: track 0.00 -> 95.7 mm
- net SW_4: track 0.00 -> 85.8 mm
- net USBC.D+: track 0.00 -> 77.1 mm, vias 0 -> 1
- net USBC.D-: track 0.00 -> 75.3 mm, vias 0 -> 1
- net I2C_SCL: track 0.00 -> 65.3 mm
- net I2C_SDA: track 0.00 -> 52.2 mm
- net PB_0: track 0.00 -> 41.9 mm
- net PB_1: track 0.00 -> 36.8 mm
- net PB_3: track 0.00 -> 32.0 mm
- net PB_2: track 0.00 -> 23.8 mm
- net LED_3: track 0.00 -> 19.9 mm
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- added copper zone on layer 2, net GND
- added copper zone on layer 15, net VDD_3P3V
- added copper zone on layer 1, net VDD_5V
Other:
- board outline added: 69.8 x 114.3 mm
- board text added: "ENGI301 Arcade Machine"
- board text added: "Game Selector"
- board text added: "Rev 1A"
- board text added: "USB Port"
