File: project_02/ArcadeMachine.sch (EAGLE design)
At the start: 5 parts, among them U1 POCKETBEAGLE, U2 0.56_HEX_BACKPACK, U3 BUZZER

Commit message: Finished project
Parts:
- added C1: 1uF, ArcadeMachine:SPARKFUN-CAPACITORS_CAP0603-CAP
- added FUD1, FUD2, FUD3: FIDUCIAL, ArcadeMachine:FIDUCIAL
- added R3, R4, R5, R6: 1K, ArcadeMachine:R_R0603
- added SW1, SW2, SW3, SW4: LED_TACTILE_BUTTON, ArcadeMachine:LED_TACTILE_BUTTON
- added SW5: ROTARY_SWITCH, ArcadeMachine:ROTARY_SWITCH
- added U4: TPD4S012_DRY_6, ArcadeMachine:TPD4S012_DRY_6
- added X1: (no value), ArcadeMachine:GHI2_USB_HOST_W/CHASSIS_GND
Connections:
- new net BUZZER: U1.GPIO47, U3.+
- new net LED_0: SW1.5, U1.PRU0.3
- new net LED_1: SW2.5, U1.GPIO64
- new net LED_2: SW3.5, U1.PRU0.5
- new net LED_3: SW4.5, U1.GPIO44
- new net PB_0: R3.1, SW1.1, SW1.3, U1.PRU0.6
- new net PB_1: R4.1, SW2.1, SW2.3, U1.GPIO65
- new net PB_2: R6.1, SW3.1, SW3.3, U1.PRU0.2
- new net PB_3: R5.1, SW4.1, SW4.3, U1.GPIO46
- new net SW_0: SW5.1, U1.GPIO58
- new net SW_1: SW5.2, U1.GPIO57
- new net SW_2: SW5.3, U1.GPIO60
- new net SW_3: SW5.4, U1.GPIO52
- new net SW_4: SW5.5, U1.GPIO59
- new net USBC.D+: U1.USB1.D-, U4.D-, X1.D+
- new net USBC.D-: U1.USB1.D+, U4.D+, X1.D-
- new net USB_DC: C1.1, U4.VBUS, X1.VBUS
- net GND: now also C1.2, SW1.2, SW1.4, SW1.6, SW2.2, SW2.4, SW2.6, SW3.2, SW3.4, SW3.6, SW4.2, SW4.4, SW4.6, SW5.C, U3.-, U4.GND, X1.GND
- net VDD_3P3V: now also R3.2, R4.2, R5.2, R6.2
- net VDD_5V: no longer U1.VOUT@2
Other:
- note added: "Buzzer"
- note added: "Game Selection"
- note added: "Light-Up Buttons"
- note added: "PocketBeagle"
- note added: "Screen"
- note added: "USB Port"
- moved on the sheet: R1, R2, U1, U2, U3
